Commit message: fixing gazebo 7 bug

File: cob_gazebo_objects/objects/bookcase.urdf.xacro (robot description, xacro)
@@ -33,11 +33,11 @@
 			<origin xyz="0 0 0" />
 			<geometry>
-				<box size="0.00 0.00 0.00" />
-			</geometry>
-		</visual>
-		<collision>
-			<origin xyz="0 0 0" />
-			<geometry>
-				<box size="0.00 0.00 0.00" />
+				<box size="0.01 0.01 0.01" />
+			</geometry>
+		</visual>
+		<collision>
+			<origin xyz="0 0 0" />
+			<geometry>
+				<box size="0.01 0.01 0.01" />
 			</geometry>
 		</collision>

File: cob_gazebo_objects/objects/cabinet.urdf.xacro (robot description, xacro)
@@ -30,5 +30,5 @@
 			<origin xyz="0 0 0" />
 			<geometry>
-				<box size="0.00 0.00 0.00" />
+				<box size="0.10 0.10 0.10" />
 			</geometry>
 		</collision>

File: cob_gazebo_objects/objects/couch.urdf.xacro (robot description, xacro)
@@ -22,5 +22,5 @@
 			<origin xyz="0 0 0" />
 			<geometry>
-				<box size="0.00 0.00 0.00" />
+				<box size="0.10 0.10 0.10" />
 			</geometry>
 		</collision>

File: cob_gazebo_objects/objects/tv_samsung.urdf (robot description, URDF)
Before this commit: robot my_object, 1 links, 0 joints
Links:
- link base_link: geometry collision box size=0.99 0.10 0.67; visual mesh filename=package://cob_gazebo_objects/Media/models/tv_samsung.dae
